File: kicad/battery_checker.kicad_sch (KiCad schematic)
At the start: 21 parts, among them J1 AVRISPmkII, SW1 POWER, U1 ATtiny13A

Commit message: update README
Connections:
- net ADCEN is gone; now on net ~{ADCEN}: D5.2 (A), U1.3 (PB4)
Other:
- note added: "Additional Circuit 追加の回路"
- note added: "Original Circuit オリジナルの回路"
- note removed: "ADDITIONAL CIRCUIT"
- moved on the sheet: D6, D7, D8, J1, R6, R7, R8
